Commit message: openAI gym humanoid fixes

File: urdf/one_thumb.urdf.xacro (robot description, xacro)
@@ -13,4 +13,13 @@
       </material>
     </visual>
+    <collision>
+      <geometry>
+        <mesh filename="package://ros2_galactic_urdf_finger/thumb_metacarpal_joint.dae"/>
+      </geometry>
+    </collision>
+    <inertial>
+      <mass value="0.01"/>
+      <inertia ixx="0.4" ixy="0.0" ixz="0.0" iyy="0.4" iyz="0.0" izz="0.2"/>
+    </inertial>
   </link>
   <link name="${prefix}_metacarpals_2">
@@ -24,4 +33,13 @@
       </material>
     </visual>
+    <collision>
+      <geometry>
+        <mesh filename="package://ros2_galactic_urdf_finger/metacarpals_joint.dae"/>
+      </geometry>
+    </collision>
+    <inertial>
+      <mass value="0.01"/>
+      <inertia ixx="0.4" ixy="0.0" ixz="0.0" iyy="0.4" iyz="0.0" izz="0.2"/>
+    </inertial>
   </link>
   <link name="${prefix}_proximal">
@@ -35,4 +53,13 @@
       </material>
     </visual>
+    <collision>
+      <geometry>
+        <mesh filename="package://ros2_galactic_urdf_finger/proximal.dae"/>
+      </geometry>
+    </collision>
+    <inertial>
+      <mass value="0.01"/>
+      <inertia ixx="0.4" ixy="0.0" ixz="0.0" iyy="0.4" iyz="0.0" izz="0.2"/>
+    </inertial>
   </link>
   <link name="${prefix}_intermediate">
@@ -46,4 +73,13 @@
       </material>
     </visual>
+    <collision>
+      <geometry>
+        <mesh filename="package://ros2_galactic_urdf_finger/intermediate.dae"/>
+      </geometry>
+    </collision>
+    <inertial>
+      <mass value="0.01"/>
+      <inertia ixx="0.4" ixy="0.0" ixz="0.0" iyy="0.4" iyz="0.0" izz="0.2"/>
+    </inertial>
   </link>
   <link name="${prefix}_distal">
@@ -57,4 +93,13 @@
       </material>
     </visual>
+    <collision>
+      <geometry>
+        <mesh filename="package://ros2_galactic_urdf_finger/distal.dae"/>
+      </geometry>
+    </collision>
+    <inertial>
+      <mass value="0.01"/>
+      <inertia ixx="0.4" ixy="0.0" ixz="0.0" iyy="0.4" iyz="0.0" izz="0.2"/>
+    </inertial>
   </link>
   <joint name="${prefix}_metacarpals_joint" type="revolute">
