Commit message: openAI humanoid fixes

File: urdf/openAIgymHumanoid2.urdf.xacro (robot description, xacro)
@@ -5,5 +5,5 @@
   <link name="${prefix}_openAIgymHumanoid_base">
     <visual>
-      <origin xyz="0 0 0.0" rpy="0 0 0" />
+      <origin xyz="0 0 0.0" rpy="0 0 1.6" />
       <geometry>
         <mesh filename="package://ros2_galactic_urdf_finger/openAIgymHumanoid_motor_base.dae"/>
@@ -163,5 +163,5 @@
     </inertial>
   </link>
-   <link name="${prefix}_proximal_l">
+  <link name="${prefix}_proximal_l">
     <visual>
       <origin xyz="0 0 -0.004" rpy="0 0 0" />
@@ -224,5 +224,5 @@
   </link>
   <joint name="${prefix}_openAIgymHumanoid_base_joint" type="fixed">
-    <origin xyz="0 -0.01 0.015" rpy="0 0 0"/>
+    <origin xyz="0 0 0.015" rpy="0 0 0"/>
     <parent link="${prefix}_openAIgymHumanoid_base"/>
     <child link="${prefix}_metacarpals"/>
@@ -262,5 +262,5 @@
   </joint>
   <joint name="${prefix}_metacarpals_joint_l" type="revolute">
-    <origin xyz="0 0 0.016" rpy="0 0 0"/>
+    <origin xyz="0 0.01 0.016" rpy="0 0 0"/>
     <parent link="${prefix}_metacarpals_l"/>
     <child link="${prefix}_metacarpals_2_l"/>
@@ -282,5 +282,5 @@
     <limit effort="30" velocity="1.0" lower="-1.6" upper="1.6" />
   </joint>
-   <joint name="${prefix}_intermediate_joint_l" type="revolute">
+  <joint name="${prefix}_intermediate_joint_l" type="revolute">
     <origin xyz="0 0 0.04" rpy="0 0 0"/>
     <parent link="${prefix}_intermediate_l"/>
