Commit message: one hand

File: urdf/one_hand.urdf.xacro (robot description, xacro)
@@ -16,4 +16,7 @@
   </link>
   </xacro:macro>
+  <xacro:phalanx name="${prefix}_base" mesh_file="package://ros2_galactic_urdf_finger/one_hand_base.dae">
+  	<origin xyz="0 0 0.0" rpy="0 0 0" />
+  </xacro:phalanx>
   <xacro:phalanx name="${prefix}_metacarpals" mesh_file="package://ros2_galactic_urdf_finger/metacarpals.dae">
   	<origin xyz="0 0 0.0" rpy="0 0 0" />
@@ -40,4 +43,7 @@
     </joint>
   </xacro:macro>
+  <xacro:phalanx_joint name="${prefix}_base_joint" parent="${prefix}_base" child="${prefix}_metacarpals">
+  	<origin xyz="0 0 0.01" rpy="0 0 0"/>
+  </xacro:phalanx_joint>
   <xacro:phalanx_joint name="${prefix}_metacarpals_joint" parent="${prefix}_metacarpals" child="${prefix}_metacarpals_2">
   	<origin xyz="0 0 0.076" rpy="0 0 0"/>

Commit message: one_hand second finger

File: urdf/one_hand.urdf.xacro (robot description, xacro)
@@ -34,4 +34,19 @@
   	<origin xyz="0 0 -0.004" rpy="0 0 0" />
   </xacro:phalanx>
+  <xacro:phalanx name="${prefix}_middle_metacarpals" mesh_file="package://ros2_galactic_urdf_finger/metacarpals.dae">
+  	<origin xyz="0 0 0.0" rpy="0 0 0" />
+  </xacro:phalanx>
+  <xacro:phalanx name="${prefix}_middle_metacarpals_2" mesh_file="package://ros2_galactic_urdf_finger/metacarpals_joint.dae">
+  	<origin xyz="0 0 -0.004" rpy="0 0 1.6" />
+  </xacro:phalanx>
+  <xacro:phalanx name="${prefix}_middle_proximal" mesh_file="package://ros2_galactic_urdf_finger/proximal.dae">
+  	<origin xyz="0 0 -0.004" rpy="0 0 0" />
+  </xacro:phalanx>
+  <xacro:phalanx name="${prefix}_middle_intermediate" mesh_file="package://ros2_galactic_urdf_finger/intermediate.dae">
+  	<origin xyz="0 0 -0.004" rpy="0 0 0" />
+  </xacro:phalanx>
+  <xacro:phalanx name="${prefix}_middle_distal" mesh_file="package://ros2_galactic_urdf_finger/distal.dae">
+  	<origin xyz="0 0 -0.004" rpy="0 0 0" />
+  </xacro:phalanx>
   <xacro:macro name="phalanx_joint" params="name parent child *origin">
     <joint name="${name}" type="revolute">
@@ -58,3 +73,18 @@
   	<origin xyz="0 0 0.04" rpy="0 0 0"/>
   </xacro:phalanx_joint>
+  <xacro:phalanx_joint name="${prefix}_middle_base_joint" parent="${prefix}_base" child="${prefix}_middle_metacarpals">
+  	<origin xyz="0 0.01 0.01" rpy="0 0 0"/>
+  </xacro:phalanx_joint>
+  <xacro:phalanx_joint name="${prefix}_middle_metacarpals_joint" parent="${prefix}_middle_metacarpals" child="${prefix}_middle_metacarpals_2">
+  	<origin xyz="0 0 0.076" rpy="0 0 0"/>
+  </xacro:phalanx_joint>
+  <xacro:phalanx_joint name="${prefix}_middle_metacarpals_2_joint" parent="${prefix}_middle_metacarpals_2" child="${prefix}_middle_proximal">
+  	<origin xyz="0 0 0.011" rpy="0 0 0"/>
+  </xacro:phalanx_joint>
+  <xacro:phalanx_joint name="${prefix}_middle_proximal_joint" parent="${prefix}_middle_proximal" child="${prefix}_middle_intermediate">
+  	<origin xyz="0 0 0.04" rpy="0 0 0"/>
+  </xacro:phalanx_joint>
+  <xacro:phalanx_joint name="${prefix}_middle_intermediate_joint" parent="${prefix}_middle_intermediate" child="${prefix}_middle_distal">
+  	<origin xyz="0 0 0.04" rpy="0 0 0"/>
+  </xacro:phalanx_joint>
 </robot>

Commit message: one_hand third finger

File: urdf/one_hand.urdf.xacro (robot description, xacro)
@@ -49,4 +49,19 @@
   	<origin xyz="0 0 -0.004" rpy="0 0 0" />
   </xacro:phalanx>
+  <xacro:phalanx name="${prefix}_ring_metacarpals" mesh_file="package://ros2_galactic_urdf_finger/metacarpals.dae">
+  	<origin xyz="0 0 0.0" rpy="0 0 0" />
+  </xacro:phalanx>
+  <xacro:phalanx name="${prefix}_ring_metacarpals_2" mesh_file="package://ros2_galactic_urdf_finger/metacarpals_joint.dae">
+  	<origin xyz="0 0 -0.004" rpy="0 0 1.6" />
+  </xacro:phalanx>
+  <xacro:phalanx name="${prefix}_ring_proximal" mesh_file="package://ros2_galactic_urdf_finger/proximal.dae">
+  	<origin xyz="0 0 -0.004" rpy="0 0 0" />
+  </xacro:phalanx>
+  <xacro:phalanx name="${prefix}_ring_intermediate" mesh_file="package://ros2_galactic_urdf_finger/intermediate.dae">
+  	<origin xyz="0 0 -0.004" rpy="0 0 0" />
+  </xacro:phalanx>
+  <xacro:phalanx name="${prefix}_ring_distal" mesh_file="package://ros2_galactic_urdf_finger/distal.dae">
+  	<origin xyz="0 0 -0.004" rpy="0 0 0" />
+  </xacro:phalanx>
   <xacro:macro name="phalanx_joint" params="name parent child *origin">
     <joint name="${name}" type="revolute">
@@ -88,3 +103,18 @@
   	<origin xyz="0 0 0.04" rpy="0 0 0"/>
   </xacro:phalanx_joint>
+  <xacro:phalanx_joint name="${prefix}_ring_base_joint" parent="${prefix}_base" child="${prefix}_ring_metacarpals">
+  	<origin xyz="0 0.02 0.01" rpy="0 0 0"/>
+  </xacro:phalanx_joint>
+  <xacro:phalanx_joint name="${prefix}_ring_metacarpals_joint" parent="${prefix}_ring_metacarpals" child="${prefix}_ring_metacarpals_2">
+  	<origin xyz="0 0 0.076" rpy="0 0 0"/>
+  </xacro:phalanx_joint>
+  <xacro:phalanx_joint name="${prefix}_ring_metacarpals_2_joint" parent="${prefix}_ring_metacarpals_2" child="${prefix}_ring_proximal">
+  	<origin xyz="0 0 0.011" rpy="0 0 0"/>
+  </xacro:phalanx_joint>
+  <xacro:phalanx_joint name="${prefix}_ring_proximal_joint" parent="${prefix}_ring_proximal" child="${prefix}_ring_intermediate">
+  	<origin xyz="0 0 0.04" rpy="0 0 0"/>
+  </xacro:phalanx_joint>
+  <xacro:phalanx_joint name="${prefix}_ring_intermediate_joint" parent="${prefix}_ring_intermediate" child="${prefix}_ring_distal">
+  	<origin xyz="0 0 0.04" rpy="0 0 0"/>
+  </xacro:phalanx_joint>
 </robot>

Commit message: one_hand fourth finger

File: urdf/one_hand.urdf.xacro (robot description, xacro)
@@ -64,4 +64,19 @@
   	<origin xyz="0 0 -0.004" rpy="0 0 0" />
   </xacro:phalanx>
+  <xacro:phalanx name="${prefix}_pinky_metacarpals" mesh_file="package://ros2_galactic_urdf_finger/metacarpals.dae">
+  	<origin xyz="0 0 0.0" rpy="0 0 0" />
+  </xacro:phalanx>
+  <xacro:phalanx name="${prefix}_pinky_metacarpals_2" mesh_file="package://ros2_galactic_urdf_finger/metacarpals_joint.dae">
+  	<origin xyz="0 0 -0.004" rpy="0 0 1.6" />
+  </xacro:phalanx>
+  <xacro:phalanx name="${prefix}_pinky_proximal" mesh_file="package://ros2_galactic_urdf_finger/proximal.dae">
+  	<origin xyz="0 0 -0.004" rpy="0 0 0" />
+  </xacro:phalanx>
+  <xacro:phalanx name="${prefix}_pinky_intermediate" mesh_file="package://ros2_galactic_urdf_finger/intermediate.dae">
+  	<origin xyz="0 0 -0.004" rpy="0 0 0" />
+  </xacro:phalanx>
+  <xacro:phalanx name="${prefix}_pinky_distal" mesh_file="package://ros2_galactic_urdf_finger/distal.dae">
+  	<origin xyz="0 0 -0.004" rpy="0 0 0" />
+  </xacro:phalanx>
   <xacro:macro name="phalanx_joint" params="name parent child *origin">
     <joint name="${name}" type="revolute">
@@ -118,3 +133,18 @@
   	<origin xyz="0 0 0.04" rpy="0 0 0"/>
   </xacro:phalanx_joint>
+  <xacro:phalanx_joint name="${prefix}_pinky_base_joint" parent="${prefix}_base" child="${prefix}_pinky_metacarpals">
+  	<origin xyz="0 -0.01 0.01" rpy="0 0 0"/>
+  </xacro:phalanx_joint>
+  <xacro:phalanx_joint name="${prefix}_pinky_metacarpals_joint" parent="${prefix}_pinky_metacarpals" child="${prefix}_pinky_metacarpals_2">
+  	<origin xyz="0 0 0.076" rpy="0 0 0"/>
+  </xacro:phalanx_joint>
+  <xacro:phalanx_joint name="${prefix}_pinky_metacarpals_2_joint" parent="${prefix}_pinky_metacarpals_2" child="${prefix}_pinky_proximal">
+  	<origin xyz="0 0 0.011" rpy="0 0 0"/>
+  </xacro:phalanx_joint>
+  <xacro:phalanx_joint name="${prefix}_pinky_proximal_joint" parent="${prefix}_pinky_proximal" child="${prefix}_pinky_intermediate">
+  	<origin xyz="0 0 0.04" rpy="0 0 0"/>
+  </xacro:phalanx_joint>
+  <xacro:phalanx_joint name="${prefix}_pinky_intermediate_joint" parent="${prefix}_pinky_intermediate" child="${prefix}_pinky_distal">
+  	<origin xyz="0 0 0.04" rpy="0 0 0"/>
+  </xacro:phalanx_joint>
 </robot>

Commit message: name fixes

File: urdf/one_hand.urdf.xacro (robot description, xacro)
@@ -88,21 +88,21 @@
     </joint>
   </xacro:macro>
-  <xacro:phalanx_joint name="${prefix}_base_joint" parent="${prefix}_base" child="${prefix}_metacarpals">
-  	<origin xyz="0 0 0.01" rpy="0 0 0"/>
+  <xacro:phalanx_joint name="${prefix}_index_base_joint" parent="${prefix}_base" child="${prefix}_metacarpals">
+  	<origin xyz="0 -0.01 0.01" rpy="0.1 0 0"/>
   </xacro:phalanx_joint>
-  <xacro:phalanx_joint name="${prefix}_metacarpals_joint" parent="${prefix}_metacarpals" child="${prefix}_metacarpals_2">
+  <xacro:phalanx_joint name="${prefix}_index_metacarpals_joint" parent="${prefix}_metacarpals" child="${prefix}_metacarpals_2">
   	<origin xyz="0 0 0.076" rpy="0 0 0"/>
   </xacro:phalanx_joint>
-  <xacro:phalanx_joint name="${prefix}_metacarpals_2_joint" parent="${prefix}_metacarpals_2" child="${prefix}_proximal">
+  <xacro:phalanx_joint name="${prefix}_index_metacarpals_2_joint" parent="${prefix}_metacarpals_2" child="${prefix}_proximal">
   	<origin xyz="0 0 0.011" rpy="0 0 0"/>
   </xacro:phalanx_joint>
-  <xacro:phalanx_joint name="${prefix}_proximal_joint" parent="${prefix}_proximal" child="${prefix}_intermediate">
+  <xacro:phalanx_joint name="${prefix}_index_proximal_joint" parent="${prefix}_proximal" child="${prefix}_intermediate">
   	<origin xyz="0 0 0.04" rpy="0 0 0"/>
   </xacro:phalanx_joint>
-  <xacro:phalanx_joint name="${prefix}_intermediate_joint" parent="${prefix}_intermediate" child="${prefix}_distal">
+  <xacro:phalanx_joint name="${prefix}_index_intermediate_joint" parent="${prefix}_intermediate" child="${prefix}_distal">
   	<origin xyz="0 0 0.04" rpy="0 0 0"/>
   </xacro:phalanx_joint>
   <xacro:phalanx_joint name="${prefix}_middle_base_joint" parent="${prefix}_base" child="${prefix}_middle_metacarpals">
-  	<origin xyz="0 0.01 0.01" rpy="0 0 0"/>
+  	<origin xyz="0 0.0 0.01" rpy="0 0 0"/>
   </xacro:phalanx_joint>
   <xacro:phalanx_joint name="${prefix}_middle_metacarpals_joint" parent="${prefix}_middle_metacarpals" child="${prefix}_middle_metacarpals_2">
@@ -119,5 +119,5 @@
   </xacro:phalanx_joint>
   <xacro:phalanx_joint name="${prefix}_ring_base_joint" parent="${prefix}_base" child="${prefix}_ring_metacarpals">
-  	<origin xyz="0 0.02 0.01" rpy="0 0 0"/>
+  	<origin xyz="0 0.01 0.01" rpy="-0.1 0 0"/>
   </xacro:phalanx_joint>
   <xacro:phalanx_joint name="${prefix}_ring_metacarpals_joint" parent="${prefix}_ring_metacarpals" child="${prefix}_ring_metacarpals_2">
@@ -134,5 +134,5 @@
   </xacro:phalanx_joint>
   <xacro:phalanx_joint name="${prefix}_pinky_base_joint" parent="${prefix}_base" child="${prefix}_pinky_metacarpals">
-  	<origin xyz="0 -0.01 0.01" rpy="0 0 0"/>
+  	<origin xyz="0 0.02 0.01" rpy="-0.2 0 0"/>
   </xacro:phalanx_joint>
   <xacro:phalanx_joint name="${prefix}_pinky_metacarpals_joint" parent="${prefix}_pinky_metacarpals" child="${prefix}_pinky_metacarpals_2">

Commit message: name fixes, add axis to xacro

File: urdf/one_hand.urdf.xacro (robot description, xacro)
@@ -79,10 +79,25 @@
   	<origin xyz="0 0 -0.004" rpy="0 0 0" />
   </xacro:phalanx>
-  <xacro:macro name="phalanx_joint" params="name parent child *origin">
+  <xacro:phalanx name="${prefix}_thumb_metacarpals" mesh_file="package://ros2_galactic_urdf_finger/thumb_metacarpal_joint.dae">
+  	<origin xyz="0 0 0.0" rpy="0 0 0" />
+  </xacro:phalanx>
+  <xacro:phalanx name="${prefix}_thumb_metacarpals_2" mesh_file="package://ros2_galactic_urdf_finger/metacarpals_joint.dae">
+  	<origin xyz="0 0 -0.004" rpy="0 0 1.6" />
+  </xacro:phalanx>
+  <xacro:phalanx name="${prefix}_thumb_proximal" mesh_file="package://ros2_galactic_urdf_finger/proximal.dae">
+  	<origin xyz="0 0 -0.004" rpy="0 0 0" />
+  </xacro:phalanx>
+  <xacro:phalanx name="${prefix}_thumb_intermediate" mesh_file="package://ros2_galactic_urdf_finger/intermediate.dae">
+  	<origin xyz="0 0 -0.004" rpy="0 0 0" />
+  </xacro:phalanx>
+  <xacro:phalanx name="${prefix}_thumb_distal" mesh_file="package://ros2_galactic_urdf_finger/distal.dae">
+  	<origin xyz="0 0 -0.004" rpy="0 0 0" />
+  </xacro:phalanx>
+  <xacro:macro name="phalanx_joint" params="name parent child *origin *axis">
     <joint name="${name}" type="revolute">
 	    <xacro:insert_block name="origin" />
 	    <parent link="${parent}"/>
 	    <child link="${child}"/>
-	    <axis xyz="0 1 0"/>
+	    <xacro:insert_block name="axis" />
 	    <limit effort="30" velocity="1.0" lower="-1.6" upper="1.6" />
     </joint>
@@ -90,61 +105,101 @@
   <xacro:phalanx_joint name="${prefix}_index_base_joint" parent="${prefix}_base" child="${prefix}_metacarpals">
   	<origin xyz="0 -0.01 0.01" rpy="0.1 0 0"/>
+  	<axis xyz="0 1 0"/>
   </xacro:phalanx_joint>
   <xacro:phalanx_joint name="${prefix}_index_metacarpals_joint" parent="${prefix}_metacarpals" child="${prefix}_metacarpals_2">
   	<origin xyz="0 0 0.076" rpy="0 0 0"/>
+  	<axis xyz="0 1 0"/>
   </xacro:phalanx_joint>
   <xacro:phalanx_joint name="${prefix}_index_metacarpals_2_joint" parent="${prefix}_metacarpals_2" child="${prefix}_proximal">
   	<origin xyz="0 0 0.011" rpy="0 0 0"/>
+  	<axis xyz="1 0 0"/>
   </xacro:phalanx_joint>
   <xacro:phalanx_joint name="${prefix}_index_proximal_joint" parent="${prefix}_proximal" child="${prefix}_intermediate">
   	<origin xyz="0 0 0.04" rpy="0 0 0"/>
+  	<axis xyz="0 1 0"/>
   </xacro:phalanx_joint>
   <xacro:phalanx_joint name="${prefix}_index_intermediate_joint" parent="${prefix}_intermediate" child="${prefix}_distal">
   	<origin xyz="0 0 0.04" rpy="0 0 0"/>
+  	<axis xyz="0 1 0"/>
   </xacro:phalanx_joint>
   <xacro:phalanx_joint name="${prefix}_middle_base_joint" parent="${prefix}_base" child="${prefix}_middle_metacarpals">
   	<origin xyz="0 0.0 0.01" rpy="0 0 0"/>
+  	<axis xyz="0 1 0"/>
   </xacro:phalanx_joint>
   <xacro:phalanx_joint name="${prefix}_middle_metacarpals_joint" parent="${prefix}_middle_metacarpals" child="${prefix}_middle_metacarpals_2">
   	<origin xyz="0 0 0.076" rpy="0 0 0"/>
+  	<axis xyz="0 1 0"/>
   </xacro:phalanx_joint>
   <xacro:phalanx_joint name="${prefix}_middle_metacarpals_2_joint" parent="${prefix}_middle_metacarpals_2" child="${prefix}_middle_proximal">
   	<origin xyz="0 0 0.011" rpy="0 0 0"/>
+  	<axis xyz="1 0 0"/>
   </xacro:phalanx_joint>
   <xacro:phalanx_joint name="${prefix}_middle_proximal_joint" parent="${prefix}_middle_proximal" child="${prefix}_middle_intermediate">
   	<origin xyz="0 0 0.04" rpy="0 0 0"/>
+  	<axis xyz="0 1 0"/>
   </xacro:phalanx_joint>
   <xacro:phalanx_joint name="${prefix}_middle_intermediate_joint" parent="${prefix}_middle_intermediate" child="${prefix}_middle_distal">
   	<origin xyz="0 0 0.04" rpy="0 0 0"/>
+  	<axis xyz="0 1 0"/>
   </xacro:phalanx_joint>
   <xacro:phalanx_joint name="${prefix}_ring_base_joint" parent="${prefix}_base" child="${prefix}_ring_metacarpals">
   	<origin xyz="0 0.01 0.01" rpy="-0.1 0 0"/>
+  	<axis xyz="0 1 0"/>
   </xacro:phalanx_joint>
   <xacro:phalanx_joint name="${prefix}_ring_metacarpals_joint" parent="${prefix}_ring_metacarpals" child="${prefix}_ring_metacarpals_2">
   	<origin xyz="0 0 0.076" rpy="0 0 0"/>
+  	<axis xyz="0 1 0"/>
   </xacro:phalanx_joint>
   <xacro:phalanx_joint name="${prefix}_ring_metacarpals_2_joint" parent="${prefix}_ring_metacarpals_2" child="${prefix}_ring_proximal">
   	<origin xyz="0 0 0.011" rpy="0 0 0"/>
+  	<axis xyz="1 0 0"/>
   </xacro:phalanx_joint>
   <xacro:phalanx_joint name="${prefix}_ring_proximal_joint" parent="${prefix}_ring_proximal" child="${prefix}_ring_intermediate">
   	<origin xyz="0 0 0.04" rpy="0 0 0"/>
+  	<axis xyz="0 1 0"/>
   </xacro:phalanx_joint>
   <xacro:phalanx_joint name="${prefix}_ring_intermediate_joint" parent="${prefix}_ring_intermediate" child="${prefix}_ring_distal">
   	<origin xyz="0 0 0.04" rpy="0 0 0"/>
+  	<axis xyz="0 1 0"/>
   </xacro:phalanx_joint>
   <xacro:phalanx_joint name="${prefix}_pinky_base_joint" parent="${prefix}_base" child="${prefix}_pinky_metacarpals">
   	<origin xyz="0 0.02 0.01" rpy="-0.2 0 0"/>
+  	<axis xyz="0 1 0"/>
   </xacro:phalanx_joint>
   <xacro:phalanx_joint name="${prefix}_pinky_metacarpals_joint" parent="${prefix}_pinky_metacarpals" child="${prefix}_pinky_metacarpals_2">
   	<origin xyz="0 0 0.076" rpy="0 0 0"/>
+  	<axis xyz="0 1 0"/>
   </xacro:phalanx_joint>
   <xacro:phalanx_joint name="${prefix}_pinky_metacarpals_2_joint" parent="${prefix}_pinky_metacarpals_2" child="${prefix}_pinky_proximal">
   	<origin xyz="0 0 0.011" rpy="0 0 0"/>
+  	<axis xyz="1 0 0"/>
   </xacro:phalanx_joint>
   <xacro:phalanx_joint name="${prefix}_pinky_proximal_joint" parent="${prefix}_pinky_proximal" child="${prefix}_pinky_intermediate">
   	<origin xyz="0 0 0.04" rpy="0 0 0"/>
+  	<axis xyz="0 1 0"/>
   </xacro:phalanx_joint>
   <xacro:phalanx_joint name="${prefix}_pinky_intermediate_joint" parent="${prefix}_pinky_intermediate" child="${prefix}_pinky_distal">
   	<origin xyz="0 0 0.04" rpy="0 0 0"/>
+  	<axis xyz="0 1 0"/>
+  </xacro:phalanx_joint>
+  <xacro:phalanx_joint name="${prefix}_thumb_base_joint" parent="${prefix}_base" child="${prefix}_thumb_metacarpals">
+  	<origin xyz="0 -0.02 0.01" rpy="0.1 0 0"/>
+  	<axis xyz="0 1 0"/>
+  </xacro:phalanx_joint>
+  <xacro:phalanx_joint name="${prefix}_thumb_metacarpals_joint" parent="${prefix}_thumb_metacarpals" child="${prefix}_thumb_metacarpals_2">
+  	<origin xyz="0 0 0.016" rpy="0 0 0"/>
+  	<axis xyz="0 1 0"/>
+  </xacro:phalanx_joint>
+  <xacro:phalanx_joint name="${prefix}_thumb_metacarpals_2_joint" parent="${prefix}_thumb_metacarpals_2" child="${prefix}_thumb_proximal">
+  	<origin xyz="0 0 0.011" rpy="0 0 0"/>
+  	<axis xyz="1 0 0"/>
+  </xacro:phalanx_joint>
+  <xacro:phalanx_joint name="${prefix}_thumb_proximal_joint" parent="${prefix}_thumb_proximal" child="${prefix}_thumb_intermediate">
+  	<origin xyz="0 0 0.04" rpy="0 0 0"/>
+  	<axis xyz="0 1 0"/>
+  </xacro:phalanx_joint>
+  <xacro:phalanx_joint name="${prefix}_thumb_intermediate_joint" parent="${prefix}_thumb_intermediate" child="${prefix}_thumb_distal">
+  	<origin xyz="0 0 0.04" rpy="0 0 0"/>
+  	<axis xyz="0 1 0"/>
   </xacro:phalanx_joint>
 </robot>

Commit message: fixes

File: urdf/one_hand.urdf.xacro (robot description, xacro)
@@ -184,5 +184,5 @@
   </xacro:phalanx_joint>
   <xacro:phalanx_joint name="${prefix}_thumb_base_joint" parent="${prefix}_base" child="${prefix}_thumb_metacarpals">
-  	<origin xyz="0 -0.02 0.01" rpy="0.1 0 0"/>
+  	<origin xyz="0 -0.02 0.01" rpy="0.7 0 0.8"/>
   	<axis xyz="0 1 0"/>
   </xacro:phalanx_joint>
